Commit message: Added and tuned navigation stack for RangerX platform.  More tuning needed, but is functional for simple navigation and obstacle avoidance.

File: robot_odometry/URDF/rangerX.urdf (robot description, URDF)
Before this commit: robot rangerX, 2 links, 1 joints
Joints:
- joint base_to_laser: origin xyz=0 0 1.45 rpy=0 0 -1.57 -> xyz=-0.065 0 1.41 rpy=0 0 -1.57
